Commit message: Improbed valve URDF

File: source/isaaclab_so100/isaaclab_so100/tasks/manager_based/isaaclab_so100/asset/valve/valve.urdf (robot description, URDF)
Before this commit: robot valve, 2 links, 1 joints
Links:
- added link sphere_1, mass 0.01; collision sphere radius=0.01; visual sphere radius=0.01
- added link sphere_2, mass 0.01; collision sphere radius=0.01; visual sphere radius=0.01
- added link sphere_3, mass 0.01; collision sphere radius=0.01; visual sphere radius=0.01
- added link sphere_4, mass 0.01; collision sphere radius=0.01; visual sphere radius=0.01
- added link valve_vertical_cylinder, mass 0.05; collision cylinder length=0.05 radius=0.01; visual cylinder length=0.05 radius=0.01
- link valve_base: geometry collision cylinder length=0.05 radius=0.02; visual cylinder length=0.05 radius=0.02
- link valve_handle: geometry collision cylinder length=0.20 radius=0.01; collision cylinder length=0.20 radius=0.01
Joints:
- added joint sphere_1_joint: type fixed, parent valve_handle, child sphere_1, origin xyz=0.05 0 0 rpy=0 0 0
- added joint sphere_2_joint: type fixed, parent valve_handle, child sphere_2, origin xyz=-0.05 0 0 rpy=0 0 0
- added joint sphere_3_joint: type fixed, parent valve_handle, child sphere_3, origin xyz=0 0.05 0 rpy=0 0 0
- added joint sphere_4_joint: type fixed, parent valve_handle, child sphere_4, origin xyz=0 -0.05 0 rpy=0 0 0
- added joint vertical_cylinder_joint: type fixed, parent valve_handle, child valve_vertical_cylinder, origin xyz=0 0 0 rpy=0 0 0
