Commit message: Trained agent that more less turns the valve (single env, still issues with rotation reward...

File: source/isaaclab_so100/isaaclab_so100/tasks/manager_based/isaaclab_so100/asset/valve2.urdf (robot description, URDF)
Before this commit: robot valve, 6 links, 5 joints
Links:
- link handle_end_x_neg: mass None -> 0.01; geometry collision sphere radius=0.01; visual sphere radius=0.01
- link handle_end_x_pos: mass None -> 0.01; geometry collision sphere radius=0.01; visual sphere radius=0.01
- link handle_end_y_neg: mass None -> 0.01; geometry collision sphere radius=0.01; visual sphere radius=0.01
- link handle_end_y_pos: mass None -> 0.01; geometry collision sphere radius=0.01; visual sphere radius=0.01
Joints:
- joint joint_x_neg: axis (none) -> 0 0 1; limit (none) -> lower=0 upper=0.01 effort=5 velocity=1; type fixed -> revolute
- joint joint_x_pos: axis (none) -> 0 0 1; limit (none) -> lower=0 upper=0.01 effort=5 velocity=1; type fixed -> revolute
- joint joint_y_neg: axis (none) -> 0 0 1; limit (none) -> lower=0 upper=0.01 effort=5 velocity=1; type fixed -> revolute
- joint joint_y_pos: axis (none) -> 0 0 1; limit (none) -> lower=0 upper=0.01 effort=5 velocity=1; type fixed -> revolute
